File: aduinobasic.brd (EAGLE design)
At the start: 84 parts

Commit message: .
Parts:
- added 3C10: 470µ / 10V, HWProgUSB:RCL_E3,5-8
- added 3C11: 100µ 16V, HWProgUSB:RCL_E3,5-8
- added 3C12: 100n, rcl:C1206
- added 3C8: 100n, rc-elektronik:C1206
- added 3C9: 1n, rcl:C025-025X050
- added 3D2: MC34063AD, mc34063:SOIC8
- added 3L2: 100uh, rcl:0207/10
- added 3R5: 220, rcl:M1206
- added 3R6: 0.5-1, rcl:M1206
- added 3R7: 20k, rcl:M0805
- added 3R8: 2k2, rcl:M0805
- added 3VD2: SS12, diode:SMB
- S38: value < -> ,<
- S44: value > -> .>
- turned S29 to 270 degrees
- turned S50 to 180 degrees
- turned S53 to 180 degrees
- turned S56 to 270 degrees
- turned S57 to 270 degrees
- turned S58 to 270 degrees
Connections:
- new net D12: S16.1, S3.1, S37.1, S54.1, S8.1, S9.1, S9.2
- new net D13: S11.1, S13.1, S17.1, S43.1
- new net D14: S12.1, S19.1, S33.1, S49.1
- new net D15: S18.1, S21.1, S24.1, S29.1, S29.2, S32.1, S36.1, S36.2, S42.1, S42.2, S7.1
- new net D16: S14.1, S15.1, S20.1, S23.1, S23.2, S25.1, S35.1, S35.2, S48.1, S5.1
- new net D17: S10.1, S30.1, S39.1, S41.1, S41.2, S6.1
- new net D18: S27.1, S31.1, S44.1, S47.1
- new net D19: S26.1, S4.1, S40.1, S45.1, S45.2, S46.1, S46.2, S50.1, S50.2, S55.1, S55.2
- new net D23: S2.1, S22.1, S22.2, S28.1, S28.2, S38.1
- new net D24: S51.1, S51.2
- new net D25: S56.1, S56.2
- new net D26: S1.1, S52.1, S52.2
- new net D3: S34.1, S34.2, S53.1, S57.1, S57.2, S58.1, S58.2
- new net N$5: 3D2.8, 3R5.1
- new net N$6: 3D2.7, 3L2.1, 3R5.2, 3R6.2
- new net N$7: 3D2.5, 3R7.1, 3R8.2
- new net N$8: 3D2.1, 3L2.2, 3VD2.A
- new net N$9: 3C9.1, 3D2.3
- net +12V: now also 3C11.+, 3C12.2, 3R7.2, 3VD2.C
- net +5V: now also 3C10.+, 3C8.1, 3D2.6, 3R6.1
- net GND: now also 3C10.-, 3C11.-, 3C12.1, 3C8.2, 3C9.2, 3D2.2, 3D2.4, 3R8.1
- net U10: now also S1.3, S24.4; no longer S12.3
- net U11: now also S11.4, S12.3, S12.4, S18.4, S26.4, S30.4, S31.4
- net U4: now also S36.4, S37.4, S41.4, S43.4, S50.4; no longer S2.3, S22.3, S28.3
- net U5: now also S48.4, S55.4
- net U7: now also S16.4, S38.4, S44.4, S51.4, S57.4, S58.4
- net U8: now also S2.3, S22.3, S22.4, S28.3, S28.4
- net U9: now also S27.4, S29.4, S34.4, S40.4, S52.4, S8.4; no longer S1.3
Routing:
- net D3: track 0.00 -> 60.5 mm
- net D19: track 0.00 -> 58.5 mm
- net U9: track 83.3 -> 140.3 mm
- net U7: track 65.8 -> 108.8 mm
- net D16: track 0.00 -> 29.7 mm
- net D15: track 0.00 -> 27.7 mm
- net U8: track 0.00 -> 18.9 mm
- net D23: track 0.00 -> 15.7 mm
- net U5: track 31.2 -> 19.5 mm
- net U10: track 45.3 -> 57.0 mm
- net D24: track 0.00 -> 6.50 mm
- net D12: track 0.00 -> 6.50 mm
- net D26: track 0.00 -> 6.50 mm
- net D25: track 0.00 -> 6.50 mm
- net D17: track 0.00 -> 6.50 mm
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
Commit message: .
Parts:
- removed 3C1: 100n, rc-elektronik:C1206
- removed 3C2: 470µ / 10V, HWProgUSB:RCL_E3,5-8
- removed 3C3: 100µ 16V, HWProgUSB:RCL_E3,5-8
- removed 3C4: 1n, rcl:C025-025X050
- removed 3C5: 100n, rcl:C1206
- removed 3D1, 3D2: MC34063AD, mc34063:SOIC8
- removed 3L1: 100uh, rcl:0207/10
- removed 3R1: 0.5-1, rcl:M1206
- removed 3R2: 220, rcl:M1206
- removed 3R3: 2k2, rcl:M0805
- removed 3R4: 20k, rcl:M0805
- removed 3VD1: SS12, diode:SMB
- added DA1: MC34063AD, mc34063:SOIC8
- added JP1: (no value), pinhead:1X02
- 3C10, 3C11: device HWProgUSB:RCL_E3,5-8 -> HWProgUSB:RCL_E2-5
- 3R5: value 220 -> 180
- 3R6: value 0.5-1 -> 1
- 3R7: value 20k -> 3k
- 3R8: value 2k2 -> 1k
- C1, C2, C3: value (none) -> 100n
- Z1: value (none) -> 16Mhz
- moved 3C11 61.3 mm to (56.5, 37.5), turned to 45 degrees
- moved 3C12 60.7 mm to (55.6, 33.3), flipped to the bottom
- moved 3R8 58.5 mm to (53.7, 30.8), flipped to the bottom
- moved 3R6 54.4 mm to (53.3, 29.8), turned to 90 degrees
- moved 3R5 47.2 mm to (53.3, 34.0)
- moved 3VD2 44.5 mm to (44.8, 31.4), flipped to the bottom
- moved 3C10 44.2 mm to (30.2, 34.6), turned to 90 degrees
- moved 3R7 40.5 mm to (49.5, 32.1), flipped to the bottom, turned to 90 degrees
- moved 3C9 36.9 mm to (34.3, 28.6), turned to 270 degrees
- moved 3L2 35.3 mm to (42.5, 28.9), turned to 180 degrees
- moved 3C8 28.3 mm to (27.9, 34.6), flipped to the bottom, turned to 90 degrees
- moved PORT 0.95 mm to (44.5, 58.7), turned to 0 degrees
- moved PORT1 0.95 mm to (44.5, 61.3)
- turned S19 to 270 degrees
- turned S21 to 270 degrees
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- renumbered Q1 to Z1
Connections:
- removed net +12V: 3C11.+, 3C12.2, 3C3.+, 3C5.2, 3R4.2, 3R7.2, 3VD1.C, 3VD2.C
- removed net +5V: 3C1.1, 3C10.+, 3C2.+, 3C8.1, 3D1.6, 3D2.6, 3R1.1, 3R6.1
- removed net N$104: 3D1.8, 3R2.1
- removed net N$105: 3D1.7, 3L1.1, 3R1.2, 3R2.2
- removed net N$106: 3D1.5, 3R3.2, 3R4.1
- removed net N$107: 3D1.1, 3L1.2, 3VD1.A
- removed net N$108: 3C4.1, 3D1.3
- new net V+: 3C10.+, 3C8.1, 3R6.1, DA1.6, JP1.1
- net A0: now also PORT.11; no longer PORT.2
- net A1: now also PORT.12; no longer PORT.1
- net A2: now also PORT.8; no longer PORT.5
- net A3: now also PORT.7; no longer PORT.6
- net A6: now also PORT.9; no longer PORT.4
- net A7: now also PORT.10; no longer PORT.3
- net D0: now also PORT.6; no longer PORT.7
- net D1: now also PORT.5; no longer PORT.8
- net D12: now also S16.2, S3.2, S54.2, S8.2
- net D13: now also S11.2, S13.2, S17.2
- net D14: now also S19.2, S33.2
- net D15: now also S18.2, S21.2, S24.2, S7.2; no longer S24.1
- net D16: now also S20.2, S25.2, S5.2
- net D17: now also S30.2, S39.2, S6.2
- net D18: now also S31.2
- net D19: now also S4.2, S40.2
- net D2: now also PORT.4; no longer PORT.9
- net D23: now also S2.2
- net D26: now also S1.2
- net D3: now also S53.2
- net D4: now also PORT.3; no longer PORT.10
- net D6: now also PORT.1; no longer PORT.12
- net D7: now also PORT.2; no longer PORT.11
- net GND: now also DA1.2, DA1.4, JP1.2, PORT1.1, PORT1.10, PORT1.11, PORT1.12, PORT1.2, PORT1.3, PORT1.4, PORT1.5, PORT1.6, PORT1.7, PORT1.8, PORT1.9; no longer 3C1.2, 3C2.-, 3C3.-, 3C4.2, 3C5.1, 3D1.2, 3D1.4, 3D2.2, 3D2.4, 3R3.1
- net N$5: now also DA1.8; no longer 3D2.8
- net N$6: now also DA1.7; no longer 3D2.7
- net N$7: now also DA1.5; no longer 3D2.5
- net N$8: now also DA1.1; no longer 3D2.1
- net N$9: now also DA1.3; no longer 3D2.3
- net U10: now also S1.4, S10.4, S53.4; no longer S24.3
- net U11: now also S20.4, S9.4
- net U5: now also S3.4, S39.4
- net U6: now also S21.4
- net U7: now also S14.4, S33.4
- net U8: now also S23.4, S46.4, S54.4
- net U9: now also S13.4, S15.4, S19.4, S6.4; no longer S19.3
- net VCC: now also 3C11.+, 3C12.2, 3R7.2, 3VD2.C
Routing:
- net U8: track 18.9 -> 181.0 mm
- net D17: track 6.50 -> 139.6 mm, vias 0 -> 3
- net U10: track 57.0 -> 180.4 mm
- net U5: track 19.5 -> 129.6 mm, vias 0 -> 2
- net D26: track 6.50 -> 113.5 mm
- net D15: track 27.7 -> 118.7 mm
- net D12: track 6.50 -> 97.5 mm
- net D16: track 29.7 -> 118.8 mm
- net D13: track 0.00 -> 79.1 mm
- net GND: track 41.5 -> 115.1 mm
- net D19: track 58.5 -> 128.0 mm
- net D18: track 0.00 -> 69.2 mm
- net U11: track 81.7 -> 144.5 mm
- net U6: track 0.00 -> 53.8 mm
- net D14: track 0.00 -> 51.1 mm
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Other:
- board outline added: 111.1 x 52.4 mm

Commit message: .
Parts:
- R1: value (none) -> 10k
- renumbered JP1 to POW
Connections:
- net V+ renamed N$3
- net D18: no longer S31.1
- net U11: no longer S30.4
- net U7: no longer S44.3
- net U9: no longer S29.3
Routing:
- net D12: track 97.5 -> 141.3 mm
- net D3: track 67.0 -> 105.2 mm
- net D14: track 51.1 -> 84.5 mm
- net D16: track 118.8 -> 143.6 mm
- net D17: track 139.6 -> 117.1 mm
- net U11: track 144.5 -> 130.0 mm
- net U5: track 129.6 -> 117.8 mm
- net U8: track 181.0 -> 174.5 mm
- net U7: track 154.4 -> 147.9 mm
- net D19: track 128.0 -> 121.5 mm
- net D18: track 69.2 -> 62.7 mm
- net U9: track 167.1 -> 160.6 mm
- net GND: track 115.1 -> 111.6 mm
- net N$3: track 14.4 -> 13.5 mm

Commit message: .
Parts:
- removed 3C10: 470µ / 10V, HWProgUSB:RCL_E2-5
- removed 3C11: 100µ 16V, HWProgUSB:RCL_E2-5
- removed 3C12: 100n, rcl:C1206
- removed 3C6, 3C7, 3C9: 1n, rcl:C025-025X050
- removed 3C8: 100n, rc-elektronik:C1206
- removed 3L2: 100uh, rcl:0207/10
- removed 3R5: 180, rcl:M1206
- removed 3R6: 1, rcl:M1206
- removed 3R7: 3k, rcl:M0805
- removed 3R8: 1k, rcl:M0805
- removed 3VD2: SS12, diode:SMB
- added C10, C11: 100n, rcl:C1206
- added C12, C9: 100µ 16V, HWProgUSB:RCL_E2-5
- added C4, C5: 100n, rcl:C0805
- added C6: 1n, rcl:C025-025X050
- added C7: 100n, rc-elektronik:C1206
- added C8: 470µ / 10V, HWProgUSB:RCL_E2-5
- added HL1, HL2, HL3: (no value), led:LED5MM
- added IC1: 24LC256SN, microchip:SO-08
- added JMEM: (no value), ArduinoBASIC:1X04
- added L1: 100uh, rcl:0207/10
- added L2: (no value), rcl:0204/5
- added PINV: (no value), ArduinoBASIC:FE12
- added R10: 1, rcl:M1206
- added R11: 180, rcl:M1206
- added R12: 1k, rcl:M0805
- added R13: 3k, rcl:M0805
- added R2, R4, R6, R7, R8, R9: 10k, rcl:R0805
- added R3, R5: 10k, rcl:R1206W
- added SW1: POW, ArduinoBASIC:9077-2
- added T1, T2, T3: (no value), transistor:TO92-ECB
- added VD1: SS12, diode:SMB
- C2, C3: value 100n -> 1n; device rcl:C0805 -> rcl:C025-025X050
- moved DA1 76.0 mm to (106.4, 69.5), flipped to the bottom
- moved POW 54.6 mm to (65.7, 68.9)
- moved C2 21.9 mm to (29.5, 41.3), flipped to the top, turned to 90 degrees
- moved C1 18.4 mm to (51.4, 41.9), turned to 0 degrees
- moved C3 12.3 mm to (29.5, 47.6), flipped to the top, turned to 90 degrees
- moved KB2 2.22 mm to (32.1, 35.6)
- moved R1 0.71 mm to (47.6, 45.4)
- moved KB1 0.45 mm to (39.7, 51.8)
- renumbered PORT1 to PING
Connections:
- new net N$10: SW1.3, SW1.6
- new net N$11: HL1.K, T1.C
- new net N$12: R2.2, T1.B
- new net N$13: HL1.A, R3.1
- new net N$14: HL2.K, T2.C
- new net N$15: R4.2, T2.B
- new net N$16: HL2.A, R5.1
- new net N$17: HL3.K, T3.C
- new net N$18: R6.2, T3.B
- new net N$19: HL3.A, R7.1
- new net N$21: C10.2, C9.+, L2.1, R13.2, VD1.C
- new net N$4: POW.1, SW1.2, SW1.5
- net AREF: now also C1.2; no longer C2.2
- net D14: no longer S33.1
- net D15: no longer S21.2
- net D4: now also PORT.1, R2.1; no longer PORT.3
- net D6: now also PORT.2, R4.1; no longer PORT.1
- net D7: now also PORT.3, R6.1; no longer PORT.2
- net GND: now also C1.1, C10.1, C11.1, C12.-, C3.1, C4.2, C5.2, C6.2, C7.2, C8.-, C9.-, IC1.1, IC1.2, IC1.3, IC1.4, IC1.7, JMEM.4, R12.1, T1.E, T2.E, T3.E; no longer 3C10.-, 3C11.-, 3C12.1, 3C6.1, 3C7.1, 3C8.2, 3C9.2, 3R8.1, C1.2, C3.2
- net N$1: now also C2.2; no longer 3C6.2
- net N$2: now also C3.2; no longer 3C7.2
- net N$3: now also C7.1, C8.+, R10.1, SW1.1, SW1.4; no longer 3C10.+, 3C8.1, 3R6.1, POW.1
- net N$5: now also R11.1; no longer 3R5.1
- net N$6: now also L1.1, R10.2, R11.2; no longer 3L2.1, 3R5.2, 3R6.2
- net N$7: now also R12.2, R13.1; no longer 3R7.1, 3R8.2
- net N$8: now also L1.2, VD1.A; no longer 3L2.2, 3VD2.A
- net N$9: now also C6.1; no longer 3C9.1
- net SCL: now also IC1.5, JMEM.1, R9.1
- net SDA: now also IC1.6, JMEM.2, R8.1
- net U6: no longer S21.4
- net VCC: now also C11.2, C12.+, C4.1, C5.1, IC1.8, JMEM.3, L2.2, PINV.1, PINV.10, PINV.11, PINV.12, PINV.2, PINV.3, PINV.4, PINV.5, PINV.6, PINV.7, PINV.8, PINV.9, R3.2, R5.2, R7.2, R8.2, R9.2; no longer 3C11.+, 3C12.2, 3R7.2, 3VD2.C, C1.1, C3.1
Routing:
- net GND: track 111.6 -> 236.5 mm, vias 0 -> 1
- net VCC: track 105.6 -> 170.5 mm, vias 1 -> 3
- net SCL: track 0.00 -> 26.2 mm
- net N$21: track 0.00 -> 26.0 mm
- net N$7: track 3.19 -> 27.8 mm, vias 0 -> 2
- net N$3: track 13.5 -> 37.3 mm
- net SDA: track 0.00 -> 21.4 mm
- net D4: track 34.2 -> 46.7 mm
- net RESET: track 22.2 -> 32.2 mm
- net N$4: track 0.00 -> 8.78 mm
- net N$6: track 12.2 -> 20.6 mm
- net N$5: track 8.37 -> 14.4 mm
- net N$10: track 0.00 -> 4.58 mm
- net D7: track 12.2 -> 16.8 mm, vias 0 -> 1
- net N$17: track 0.00 -> 3.19 mm
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Other:
- board size 111.1 x 52.4 mm -> 111.8 x 60.6 mm

Commit message: .
Parts:
- removed IC1: 24LC256SN, microchip:SO-08
- added DD2: 24LC256SN, microchip:SO-08
- HL1, HL2, HL3: device led:LED5MM -> ArduinoBASIC:LED5MM
- R2: value 10k -> 1k
- moved R2 36.9 mm to (4.73, 44.4), turned to 0 degrees
- moved R3 27.8 mm to (14.6, 54.0)
- moved L2 27.5 mm to (107.6, 53.3)
- moved C7 27.5 mm to (55.2, 56.8)
- moved DISPLAY 27.5 mm to (19.7, 32.4)
- moved PING 27.5 mm to (19.7, 49.2)
- moved PINV 27.5 mm to (19.7, 51.8)
- moved R8 27.5 mm to (19.7, 20.6)
- moved C11 27.5 mm to (4.45, 22.5)
- moved C12 27.5 mm to (3.81, 19.4)
- moved C6 27.5 mm to (90.5, 57.1)
- moved KB2 27.5 mm to (7.30, 23.5)
- moved L1 27.5 mm to (81.6, 58.1)
- moved PORT 27.5 mm to (19.7, 46.7)
- moved R1 27.5 mm to (22.9, 33.3)
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Connections:
- net GND: now also DD2.1, DD2.2, DD2.3, DD2.4, DD2.7; no longer IC1.1, IC1.2, IC1.3, IC1.4, IC1.7
- net SCL: now also DD2.5; no longer IC1.5
- net SDA: now also DD2.6; no longer IC1.6
- net VCC: now also DD2.8; no longer IC1.8
Routing:
- net N$12: track 2.86 -> 19.1 mm
- net D4: track 46.7 -> 33.7 mm
- net N$26: track 0.00 -> 5.08 mm
- net N$20: track 0.00 -> 5.08 mm
- net N$25: track 0.00 -> 4.76 mm
- net N$24: track 0.00 -> 4.76 mm
- net N$28: track 0.00 -> 3.81 mm
- net N$23: track 0.00 -> 3.81 mm
- net N$27: track 0.00 -> 3.18 mm
- net N$22: track 0.00 -> 3.18 mm
- net VCC: track 170.5 -> 171.8 mm
- net GND: track 236.5 -> 237.4 mm

Commit message: .
Parts:
- added KB3, KB4: (no value), pinhead:1X01
- moved R10 0.63 mm to (59.7, 57.8)
- moved C10 0.32 mm to (103.5, 57.8)
- moved R11 0.32 mm to (64.5, 57.8), turned to 270 degrees
- renumbered T1 to VT1, T2 to VT2, T3 to VT3
Connections:
- net GND: now also KB4.1
- net VCC: now also KB3.1
Routing:
- net GND: track 237.4 -> 248.0 mm
- net U9: track 160.6 -> 167.8 mm
- net D3: track 105.2 -> 102.6 mm
- net N$6: track 20.6 -> 18.7 mm
- net D23: track 65.3 -> 63.8 mm
- net D16: track 143.6 -> 142.3 mm
- net D17: track 117.1 -> 117.8 mm
- net N$21: track 26.0 -> 26.7 mm
- net U11: track 130.0 -> 129.4 mm

Commit message: .
Parts:
- added BUZ: (no value), pinhead:1X01
- VT1, VT2, VT3: value (none) -> КТ315Б
Connections:
- net BUZ: now also BUZ.1
Routing:
- net BUZ: track 0.00 -> 2.48 mm
- net D2: track 24.2 -> 25.8 mm
- net N$2: track 10.8 -> 10.2 mm

Commit message: .
Parts:
- R11: value 180 -> 200
Changed lines of the file:
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@@
 <attribute name="VALUE" x="83.5025" y="53.5305" size="1.27" layer="28" rot="MR0"/>
 </element>
-<element name="R11" library="rcl" package="M1206" value="180" x="64.4525" y="57.785" smashed="yes" rot="MR270">
+<element name="R11" library="rcl" package="M1206" value="200" x="64.4525" y="57.785" smashed="yes" rot="MR270">
 <attribute name="NAME" x="66.9925" y="59.055" size="1.27" layer="26" rot="MR270"/>
 <attribute name="VALUE" x="66.9925" y="59.055" size="1.27" layer="28" rot="MR270"/>
