File: aduinobasic.brd (EAGLE design)
At the start: 111.8 x 60.6 mm, 109 parts, among them SW1 POW

Commit message: .
Parts:
- C8: value 470µ / 10V -> 47µ/16V
Changed lines of the file:
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@@
 </element>
 <element name="C6" library="rcl" package="C025-025X050" value="1n" x="90.4875" y="57.15"/>
-<element name="C8" library="HWProgUSB" package="RCL_E2-5" value="470µ / 10V" x="53.0225" y="56.8325" smashed="yes" rot="R270">
+<element name="C8" library="HWProgUSB" package="RCL_E2-5" value="47µ/16V" x="53.0225" y="56.8325" smashed="yes" rot="R270">
 <attribute name="NAME" x="52.07" y="59.436" size="1.27" layer="25" ratio="10"/>
 <attribute name="VALUE" x="50.8635" y="54.2925" size="1.27" layer="27" ratio="10" rot="R270"/>

Commit message: .
Parts:
- HL1: value (none) -> red
- HL2: value (none) -> yellow
- HL3: value (none) -> green
- R2: value 1k -> 10k
- R3: value 10k -> 300*
- R5: value 10k -> 3.3k*
- R7: value 10k -> 680*
Changed lines of the file:
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@@
 </element>
 <element name="JMEM" library="ArduinoBASIC" package="1X04" value="" x="19.05" y="18.415"/>
-<element name="HL1" library="ArduinoBASIC" package="LED5MM" value="" x="13.6525" y="56.8325" smashed="yes" rot="R180">
+<element name="HL1" library="ArduinoBASIC" package="LED5MM" value="red" x="13.6525" y="56.8325" smashed="yes" rot="R180">
 <attribute name="NAME" x="17.78" y="61.0616" size="1.27" layer="25" ratio="10" rot="R180"/>
 <attribute name="VALUE" x="10.4521" y="58.6359" size="1.27" layer="27" ratio="10" rot="R180"/>
@@
 <attribute name="VALUE" x="12.5095" y="53.975" size="1.27" layer="27" ratio="10" rot="R90"/>
 </element>
-<element name="R3" library="rcl" package="R1206W" value="10k" x="14.605" y="53.975" rot="MR270"/>
-<element name="R2" library="rcl" package="R0805" value="1k" x="4.729990625" y="44.4246" rot="MR0"/>
-<element name="HL2" library="ArduinoBASIC" package="LED5MM" value="" x="23.495" y="56.8325" smashed="yes" rot="R180">
+<element name="R3" library="rcl" package="R1206W" value="300*" x="14.605" y="53.975" rot="MR270"/>
+<element name="R2" library="rcl" package="R0805" value="10k" x="4.729990625" y="44.4246" rot="MR0"/>
+<element name="HL2" library="ArduinoBASIC" package="LED5MM" value="yellow" x="23.495" y="56.8325" smashed="yes" rot="R180">
 <attribute name="NAME" x="27.94" y="61.0616" size="1.27" layer="25" ratio="10" rot="R180"/>
 <attribute name="VALUE" x="20.2946" y="58.6359" size="1.27" layer="27" ratio="10" rot="R180"/>
@@
 <attribute name="VALUE" x="22.352" y="53.975" size="1.27" layer="27" ratio="10" rot="R90"/>
 </element>
-<element name="R5" library="rcl" package="R1206W" value="10k" x="24.765" y="53.975" rot="MR270"/>
+<element name="R5" library="rcl" package="R1206W" value="3.3k*" x="24.765" y="53.975" rot="MR270"/>
 <element name="R4" library="rcl" package="R0805" value="10k" x="15.24" y="59.055" rot="MR180"/>
-<element name="HL3" library="ArduinoBASIC" package="LED5MM" value="" x="33.3375" y="56.8325" smashed="yes" rot="R180">
+<element name="HL3" library="ArduinoBASIC" package="LED5MM" value="green" x="33.3375" y="56.8325" smashed="yes" rot="R180">
 <attribute name="NAME" x="38.4175" y="60.4266" size="1.27" layer="25" ratio="10" rot="R180"/>
 <attribute name="VALUE" x="30.1371" y="58.6359" size="1.27" layer="27" ratio="10" rot="R180"/>
@@
 <attribute name="VALUE" x="32.1945" y="53.975" size="1.27" layer="27" ratio="10" rot="R90"/>
 </element>
-<element name="R7" library="rcl" package="R0805" value="10k" x="32.385" y="53.975" rot="MR0"/>
+<element name="R7" library="rcl" package="R0805" value="680*" x="32.385" y="53.975" rot="MR0"/>
 <element name="R6" library="rcl" package="R0805" value="10k" x="25.0825" y="59.055" rot="MR180"/>
 <element name="L2" library="rcl" package="0204/5" value="" x="107.6325" y="53.34"/>

Commit message: .
Parts:
- C12, C9: value 100µ 16V -> 10µ 16V
- C2, C3: value 1n -> 22
- L2: value (none) -> 100uh
- VD1: value SS12 -> SS14
Changed lines of the file:
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@@
 <attribute name="VALUE" x="4.6355" y="39.6875" size="1.27" layer="27" ratio="10" rot="R270"/>
 </element>
-<element name="C2" library="rcl" package="C025-025X050" value="1n" x="4.7625" y="29.21" smashed="yes" rot="R90">
+<element name="C2" library="rcl" package="C025-025X050" value="22" x="4.7625" y="29.21" smashed="yes" rot="R90">
 <attribute name="NAME" x="3.2385" y="27.8765" size="1.27" layer="25" ratio="10" rot="R90"/>
 <attribute name="VALUE" x="7.5565" y="26.924" size="1.27" layer="27" ratio="10" rot="R90"/>
 </element>
-<element name="C3" library="rcl" package="C025-025X050" value="1n" x="4.7625" y="35.56" smashed="yes" rot="R90">
+<element name="C3" library="rcl" package="C025-025X050" value="22" x="4.7625" y="35.56" smashed="yes" rot="R90">
 <attribute name="NAME" x="3.2385" y="34.2265" size="1.27" layer="25" ratio="10" rot="R90"/>
 <attribute name="VALUE" x="7.5565" y="33.274" size="1.27" layer="27" ratio="10" rot="R90"/>
@@
 <attribute name="VALUE" x="79.3369" y="57.4675" size="1.27" layer="27" ratio="10"/>
 </element>
-<element name="VD1" library="diode" package="SMB" value="SS12" x="96.8375" y="57.785" smashed="yes" rot="MR0">
+<element name="VD1" library="diode" package="SMB" value="SS14" x="96.8375" y="57.785" smashed="yes" rot="MR0">
 <attribute name="NAME" x="103.759" y="59.309" size="1.27" layer="26" rot="MR0"/>
 <attribute name="VALUE" x="98.9965" y="54.356" size="1.27" layer="28" rot="MR0"/>
@@
 <attribute name="VALUE" x="50.8635" y="54.2925" size="1.27" layer="27" ratio="10" rot="R270"/>
 </element>
-<element name="C9" library="HWProgUSB" package="RCL_E2-5" value="100µ 16V" x="102.5525" y="54.61" smashed="yes" rot="R135">
+<element name="C9" library="HWProgUSB" package="RCL_E2-5" value="10µ 16V" x="102.5525" y="54.61" smashed="yes" rot="R135">
 <attribute name="NAME" x="108.928028125" y="55.687628125" size="1.27" layer="25" ratio="10" rot="R135"/>
 <attribute name="VALUE" x="102.283090625" y="57.93269375" size="1.27" layer="27" ratio="10" rot="R135"/>
@@
 <element name="R7" library="rcl" package="R0805" value="680*" x="32.385" y="53.975" rot="MR0"/>
 <element name="R6" library="rcl" package="R0805" value="10k" x="25.0825" y="59.055" rot="MR180"/>
-<element name="L2" library="rcl" package="0204/5" value="" x="107.6325" y="53.34"/>
-<element name="C12" library="HWProgUSB" package="RCL_E2-5" value="100µ 16V" x="3.81" y="19.3675" smashed="yes" rot="R180">
+<element name="L2" library="rcl" package="0204/5" value="100uh" x="107.6325" y="53.34"/>
+<element name="C12" library="HWProgUSB" package="RCL_E2-5" value="10µ 16V" x="3.81" y="19.3675" smashed="yes" rot="R180">
 <attribute name="NAME" x="5.08" y="23.749" size="1.27" layer="25" ratio="10" rot="R180"/>
 <attribute name="VALUE" x="1.27" y="21.5265" size="1.27" layer="27" ratio="10" rot="R180"/>
