File: aduinobasic.sch (EAGLE design)
At the start: 84 parts

Commit message: .
Parts:
- added 3C10: 470µ / 10V, HWProgUSB:RCL_CPOL-EUE3.5-8
- added 3C11: 100µ 16V, HWProgUSB:RCL_CPOL-EUE3.5-8
- added 3C12: 100n, rcl:C-EUC1206
- added 3C8: 100n, rc-elektronik:C-EUC1206
- added 3C9: 1n, rcl:C-EU025-025X050
- added 3D2: MC34063AD, mc34063:MC34063AD
- added 3L2: 100uh, rcl:L-US0207/10
- added 3R5: 220, rcl:R-EU_M1206
- added 3R6: 0.5-1, rcl:R-EU_M1206
- added 3R7: 20k, rcl:R-EU_M0805
- added 3R8: 2k2, rcl:R-EU_M0805
- added 3VD2: SS12, diode:SCHOTTKY-DIODESMD
- S38: value < -> ,<
- S44: value > -> .>
Connections:
- new net D12: S16.S, S3.S, S37.S, S54.S, S8.S, S9.S, S9.S1
- new net D13: S11.S, S13.S, S17.S, S43.S
- new net D14: S12.S, S19.S, S33.S, S49.S
- new net D15: S18.S, S21.S, S24.S, S29.S, S29.S1, S32.S, S36.S, S36.S1, S42.S, S42.S1, S7.S
- new net D16: S14.S, S15.S, S20.S, S23.S, S23.S1, S25.S, S35.S, S35.S1, S48.S, S5.S
- new net D17: S10.S, S30.S, S39.S, S41.S, S41.S1, S6.S
- new net D18: S27.S, S31.S, S44.S, S47.S
- new net D19: S26.S, S4.S, S40.S, S45.S, S45.S1, S46.S, S46.S1, S50.S, S50.S1, S55.S, S55.S1
- new net D23: S2.S, S22.S, S22.S1, S28.S, S28.S1, S38.S
- new net D24: S51.S, S51.S1
- new net D25: S56.S, S56.S1
- new net D26: S1.S, S52.S, S52.S1
- new net D3: S34.S, S34.S1, S53.S, S57.S, S57.S1, S58.S, S58.S1
- new net N$5: 3D2.DC, 3R5.1
- new net N$6: 3D2.IS, 3L2.1, 3R5.2, 3R6.2
- new net N$7: 3D2.FB, 3R7.1, 3R8.2
- new net N$8: 3D2.SWC, 3L2.2, 3VD2.A
- new net N$9: 3C9.1, 3D2.TC
- net +12V: now also 3C11.+, 3C12.2, 3R7.2, 3VD2.C
- net +5V: now also 3C10.+, 3C8.1, 3D2.VCC, 3R6.1
- net GND: now also 3C10.-, 3C11.-, 3C12.1, 3C8.2, 3C9.2, 3D2.GND, 3D2.SWE, 3R8.1
- net U10: now also S1.P, S24.P1; no longer S12.P
- net U11: now also S11.P1, S12.P, S12.P1, S18.P1, S26.P1, S30.P1, S31.P1
- net U4: now also S36.P1, S37.P1, S41.P1, S43.P1, S50.P1; no longer S2.P, S22.P, S28.P
- net U5: now also S48.P1, S55.P1
- net U7: now also S16.P1, S38.P1, S44.P1, S51.P1, S57.P1, S58.P1
- net U8: now also S2.P, S22.P, S22.P1, S28.P, S28.P1
- net U9: now also S27.P1, S29.P1, S34.P1, S40.P1, S52.P1, S8.P1; no longer S1.P
Other:
- note added: "10 26"

Commit message: .
Parts:
- removed 3C1: 100n, rc-elektronik:C-EUC1206
- removed 3C2: 470µ / 10V, HWProgUSB:RCL_CPOL-EUE3.5-8
- removed 3C3: 100µ 16V, HWProgUSB:RCL_CPOL-EUE3.5-8
- removed 3C4: 1n, rcl:C-EU025-025X050
- removed 3C5: 100n, rcl:C-EUC1206
- removed 3D1, 3D2: MC34063AD, mc34063:MC34063AD
- removed 3L1: 100uh, rcl:L-US0207/10
- removed 3R1: 0.5-1, rcl:R-EU_M1206
- removed 3R2: 220, rcl:R-EU_M1206
- removed 3R3: 2k2, rcl:R-EU_M0805
- removed 3R4: 20k, rcl:R-EU_M0805
- removed 3VD1: SS12, diode:SCHOTTKY-DIODESMD
- added DA1: MC34063AD, mc34063:MC34063AD
- added JP1: (no value), pinhead:PINHD-1X2
- 3C10, 3C11: device HWProgUSB:RCL_CPOL-EUE3.5-8 -> HWProgUSB:RCL_CPOL-EUE2-5
- 3R5: value 220 -> 180
- 3R6: value 0.5-1 -> 1
- 3R7: value 20k -> 3k
- 3R8: value 2k2 -> 1k
- C1, C2, C3: value (none) -> 100n
- PORT: OC_FARNELL (none) -> unknown; OC_NEWARK (none) -> unknown
- Z1: value (none) -> 16Mhz
- renumbered Q1 to Z1
Connections:
- removed net +12V: 3C11.+, 3C12.2, 3C3.+, 3C5.2, 3R4.2, 3R7.2, 3VD1.C, 3VD2.C
- removed net +5V: 3C1.1, 3C10.+, 3C2.+, 3C8.1, 3D1.VCC, 3D2.VCC, 3R1.1, 3R6.1
- removed net N$104: 3D1.DC, 3R2.1
- removed net N$105: 3D1.IS, 3L1.1, 3R1.2, 3R2.2
- removed net N$106: 3D1.FB, 3R3.2, 3R4.1
- removed net N$107: 3D1.SWC, 3L1.2, 3VD1.A
- removed net N$108: 3C4.1, 3D1.TC
- new net V+: 3C10.+, 3C8.1, 3R6.1, DA1.VCC, JP1.1
- net A0: now also PORT.11; no longer PORT.2
- net A1: now also PORT.12; no longer PORT.1
- net A2: now also PORT.8; no longer PORT.5
- net A3: now also PORT.7; no longer PORT.6
- net A6: now also PORT.9; no longer PORT.4
- net A7: now also PORT.10; no longer PORT.3
- net D0: now also PORT.6; no longer PORT.7
- net D1: now also PORT.5; no longer PORT.8
- net D12: now also S16.S1, S3.S1, S54.S1, S8.S1
- net D13: now also S11.S1, S13.S1, S17.S1
- net D14: now also S19.S1, S33.S1
- net D15: now also S18.S1, S21.S1, S24.S1, S7.S1; no longer S24.S
- net D16: now also S20.S1, S25.S1, S5.S1
- net D17: now also S30.S1, S39.S1, S6.S1
- net D18: now also S31.S1
- net D19: now also S4.S1, S40.S1
- net D2: now also PORT.4; no longer PORT.9
- net D23: now also S2.S1
- net D26: now also S1.S1
- net D3: now also S53.S1
- net D4: now also PORT.3; no longer PORT.10
- net D6: now also PORT.1; no longer PORT.12
- net D7: now also PORT.2; no longer PORT.11
- net GND: now also DA1.GND, DA1.SWE, JP1.2, PORT1.1, PORT1.10, PORT1.11, PORT1.12, PORT1.2, PORT1.3, PORT1.4, PORT1.5, PORT1.6, PORT1.7, PORT1.8, PORT1.9; no longer 3C1.2, 3C2.-, 3C3.-, 3C4.2, 3C5.1, 3D1.GND, 3D1.SWE, 3D2.GND, 3D2.SWE, 3R3.1
- net N$5: now also DA1.DC; no longer 3D2.DC
- net N$6: now also DA1.IS; no longer 3D2.IS
- net N$7: now also DA1.FB; no longer 3D2.FB
- net N$8: now also DA1.SWC; no longer 3D2.SWC
- net N$9: now also DA1.TC; no longer 3D2.TC
- net U10: now also S1.P1, S10.P1, S53.P1; no longer S24.P
- net U11: now also S20.P1, S9.P1
- net U5: now also S3.P1, S39.P1
- net U6: now also S21.P1
- net U7: now also S14.P1, S33.P1
- net U8: now also S23.P1, S46.P1, S54.P1
- net U9: now also S13.P1, S15.P1, S19.P1, S6.P1; no longer S19.P
- net VCC: now also 3C11.+, 3C12.2, 3R7.2, 3VD2.C

Commit message: .
Parts:
- removed JP1: (no value), pinhead:PINHD-1X2
- added POW: (no value), pinhead:PINHD-1X2
- R1: value (none) -> 10k
Connections:
- removed net V+: 3C10.+, 3C8.1, 3R6.1, DA1.VCC, JP1.1
- new net N$3: 3C10.+, 3C8.1, 3R6.1, DA1.VCC, POW.1
- net D18: no longer S31.S
- net GND: now also POW.2; no longer JP1.2
- net U11: no longer S30.P1
- net U7: no longer S44.P
- net U9: no longer S29.P
Changed lines of the file:
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@@
 <part name="P+3" library="supply1" deviceset="VCC" device=""/>
 <part name="GND6" library="supply1" deviceset="GND" device=""/>
-<part name="R1" library="rcl" deviceset="R-EU_" device="R0805"/>
+<part name="R1" library="rcl" deviceset="R-EU_" device="R0805" value="10k"/>
 <part name="P+4" library="supply1" deviceset="VCC" device=""/>
 <part name="C2" library="rcl" deviceset="C-EU" device="C0805" value="100n"/>
@@
 <part name="3C11" library="HWProgUSB" deviceset="RCL_CPOL-EU" device="E2-5" value="100µ 16V"/>
 <part name="3C12" library="rcl" deviceset="C-EU" device="C1206" value="100n"/>
-<part name="P+1" library="supply1" deviceset="V+" device=""/>
 <part name="P+6" library="supply1" deviceset="VCC" device=""/>
 <part name="PORT1" library="ArduinoBASIC" deviceset="FE12-1" device="">
@@
 <attribute name="OC_NEWARK" value="unknown"/>
 </part>
-<part name="JP1" library="pinhead" deviceset="PINHD-1X2" device=""/>
-<part name="GND1" library="supply1" deviceset="GND" device=""/>
-<part name="P+5" library="supply1" deviceset="V+" device=""/>
+<part name="POW" library="pinhead" deviceset="PINHD-1X2" device=""/>
 <part name="GND11" library="supply1" deviceset="GND" device=""/>
 </parts>
@@
 </instance>
 <instance part="3C8" gate="G$1" x="175.26" y="134.62" smashed="yes">
-<attribute name="NAME" x="173.101" y="142.494" size="1.778" layer="95" rot="R180"/>
-<attribute name="VALUE" x="173.101" y="139.954" size="1.778" layer="96" rot="R180"/>
+<attribute name="NAME" x="173.101" y="139.954" size="1.778" layer="95" rot="R180"/>
+<attribute name="VALUE" x="173.101" y="137.414" size="1.778" layer="96" rot="R180"/>
 </instance>
 <instance part="DA1" gate="G$1" x="208.28" y="149.86" smashed="yes">
@@
 <attribute name="VALUE" x="233.934" y="122.301" size="1.778" layer="96"/>
 </instance>
-<instance part="P+1" gate="1" x="175.26" y="154.94" smashed="yes">
-<attribute name="VALUE" x="177.8" y="157.48" size="1.778" layer="96" rot="R180"/>
-</instance>
 <instance part="P+6" gate="VCC" x="243.84" y="160.02" smashed="yes">
 <attribute name="VALUE" x="246.38" y="162.56" size="1.778" layer="96" rot="R180"/>
 </instance>
 <instance part="PORT1" gate="G$1" x="152.4" y="121.92" rot="R180"/>
-<instance part="JP1" gate="G$1" x="119.38" y="165.1"/>
-<instance part="GND1" gate="1" x="109.22" y="160.02"/>
-<instance part="P+5" gate="1" x="109.22" y="172.72" smashed="yes">
-<attribute name="VALUE" x="111.76" y="175.26" size="1.778" layer="96" rot="R180"/>
-</instance>
+<instance part="POW" gate="G$1" x="162.56" y="144.78" rot="MR0"/>
 <instance part="GND11" gate="1" x="142.24" y="101.6"/>
 </instances>
@@
 <wire x1="246.38" y1="88.9" x2="246.38" y2="10.16" width="0.762" layer="92"/>
 <wire x1="271.78" y1="88.9" x2="271.78" y2="10.16" width="0.762" layer="92"/>
-<wire x1="7.62" y1="88.9" x2="7.62" y2="10.16" width="0.762" layer="92"/>
+<wire x1="7.62" y1="88.9" x2="7.62" y2="35.56" width="0.762" layer="92"/>
 <wire x1="7.62" y1="88.9" x2="33.02" y2="88.9" width="0.762" layer="92"/>
 <wire x1="33.02" y1="88.9" x2="195.58" y2="88.9" width="0.762" layer="92"/>
@@
 <wire x1="180.34" y1="128.27" x2="180.34" y2="119.38" width="0.1524" layer="91"/>
 <junction x="180.34" y="119.38"/>
+<pinref part="POW" gate="G$1" pin="2"/>
+<wire x1="165.1" y1="144.78" x2="167.64" y2="144.78" width="0.1524" layer="91"/>
+<wire x1="167.64" y1="144.78" x2="167.64" y2="119.38" width="0.1524" layer="91"/>
+<wire x1="167.64" y1="119.38" x2="175.26" y2="119.38" width="0.1524" layer="91"/>
 </segment>
 <segment>
@@
 <pinref part="GND8" gate="1" pin="GND"/>
 <wire x1="215.9" y1="121.92" x2="215.9" y2="119.38" width="0.1524" layer="91"/>
-</segment>
-<segment>
-<pinref part="JP1" gate="G$1" pin="2"/>
-<wire x1="116.84" y1="165.1" x2="109.22" y2="165.1" width="0.1524" layer="91"/>
-<pinref part="GND1" gate="1" pin="GND"/>
-<wire x1="109.22" y1="165.1" x2="109.22" y2="162.56" width="0.1524" layer="91"/>
 </segment>
 <segment>
@@
 </segment>
 <segment>
-<pinref part="S29" gate="1" pin="P"/>
 <wire x1="134.62" y1="76.2" x2="139.7" y2="76.2" width="0.1524" layer="91"/>
 <label x="137.16" y="76.2" size="1.778" layer="95"/>
 <pinref part="S29" gate="1" pin="P1"/>
-<wire x1="139.7" y1="76.2" x2="142.24" y2="76.2" width="0.1524" layer="91"/>
 <wire x1="142.24" y1="73.66" x2="139.7" y2="73.66" width="0.1524" layer="91"/>
 <wire x1="139.7" y1="73.66" x2="139.7" y2="76.2" width="0.1524" layer="91"/>
@@
 </segment>
 <segment>
-<pinref part="S44" gate="1" pin="P"/>
 <wire x1="195.58" y1="38.1" x2="200.66" y2="38.1" width="0.1524" layer="91"/>
 <label x="198.12" y="38.1" size="1.778" layer="95"/>
 <pinref part="S44" gate="1" pin="P1"/>
-<wire x1="200.66" y1="38.1" x2="203.2" y2="38.1" width="0.1524" layer="91"/>
 <wire x1="203.2" y1="35.56" x2="200.66" y2="35.56" width="0.1524" layer="91"/>
 <wire x1="200.66" y1="35.56" x2="200.66" y2="38.1" width="0.1524" layer="91"/>
@@
 <wire x1="134.62" y1="63.5" x2="139.7" y2="63.5" width="0.1524" layer="91"/>
 <label x="137.16" y="63.5" size="1.778" layer="95"/>
-<pinref part="S30" gate="1" pin="P1"/>
 <wire x1="139.7" y1="63.5" x2="142.24" y2="63.5" width="0.1524" layer="91"/>
-<wire x1="142.24" y1="60.96" x2="139.7" y2="60.96" width="0.1524" layer="91"/>
 <wire x1="139.7" y1="60.96" x2="139.7" y2="63.5" width="0.1524" layer="91"/>
 </segment>
@@
 </segment>
 <segment>
-<pinref part="S31" gate="1" pin="S"/>
 <wire x1="160.02" y1="50.8" x2="154.94" y2="50.8" width="0.1524" layer="91"/>
 <label x="154.94" y="50.8" size="1.778" layer="95"/>
 <pinref part="S31" gate="1" pin="S1"/>
-<wire x1="154.94" y1="50.8" x2="152.4" y2="50.8" width="0.1524" layer="91"/>
 <wire x1="152.4" y1="48.26" x2="154.94" y2="48.26" width="0.1524" layer="91"/>
 <wire x1="154.94" y1="48.26" x2="154.94" y2="50.8" width="0.1524" layer="91"/>
@@
 </segment>
 </net>
-<net name="V+" class="0">
+<net name="N$3" class="0">
 <segment>
 <pinref part="DA1" gate="G$1" pin="VCC"/>
 <wire x1="193.04" y1="144.78" x2="180.34" y2="144.78" width="0.1524" layer="91"/>
 <wire x1="175.26" y1="144.78" x2="180.34" y2="144.78" width="0.1524" layer="91"/>
-<wire x1="175.26" y1="144.78" x2="175.26" y2="152.4" width="0.1524" layer="91"/>
 <pinref part="3R6" gate="G$1" pin="1"/>
 <wire x1="180.34" y1="144.78" x2="180.34" y2="152.4" width="0.1524" layer="91"/>
 <junction x="180.34" y="144.78"/>
 <wire x1="175.26" y1="137.16" x2="175.26" y2="144.78" width="0.1524" layer="91"/>
-<junction x="175.26" y="144.78"/>
 <pinref part="3C8" gate="G$1" pin="1"/>
 <pinref part="3C10" gate="G$1" pin="+"/>
 <wire x1="180.34" y1="135.89" x2="180.34" y2="144.78" width="0.1524" layer="91"/>
-<pinref part="P+1" gate="1" pin="V+"/>
-</segment>
-<segment>
-<pinref part="P+5" gate="1" pin="V+"/>
-<wire x1="109.22" y1="170.18" x2="109.22" y2="167.64" width="0.1524" layer="91"/>
-<pinref part="JP1" gate="G$1" pin="1"/>
-<wire x1="109.22" y1="167.64" x2="116.84" y2="167.64" width="0.1524" layer="91"/>
-</segment>
-</net>
+<pinref part="POW" gate="G$1" pin="1"/>
+<wire x1="165.1" y1="147.32" x2="175.26" y2="147.32" width="0.1524" layer="91"/>
+<wire x1="175.26" y1="147.32" x2="175.26" y2="144.78" width="0.1524" layer="91"/>
+<junction x="175.26" y="144.78"/>
+</segment>
+</net>

Commit message: .
Parts:
- removed 3C10: 470µ / 10V, HWProgUSB:RCL_CPOL-EUE2-5
- removed 3C11: 100µ 16V, HWProgUSB:RCL_CPOL-EUE2-5
- removed 3C12: 100n, rcl:C-EUC1206
- removed 3C6, 3C7, 3C9: 1n, rcl:C-EU025-025X050
- removed 3C8: 100n, rc-elektronik:C-EUC1206
- removed 3L2: 100uh, rcl:L-US0207/10
- removed 3R5: 180, rcl:R-EU_M1206
- removed 3R6: 1, rcl:R-EU_M1206
- removed 3R7: 3k, rcl:R-EU_M0805
- removed 3R8: 1k, rcl:R-EU_M0805
- removed 3VD2: SS12, diode:SCHOTTKY-DIODESMD
- added C10, C11: 100n, rcl:C-EUC1206
- added C12, C9: 100µ 16V, HWProgUSB:RCL_CPOL-EUE2-5
- added C4, C5: 100n, rcl:C-EUC0805
- added C6: 1n, rcl:C-EU025-025X050
- added C7: 100n, rc-elektronik:C-EUC1206
- added C8: 470µ / 10V, HWProgUSB:RCL_CPOL-EUE2-5
- added HL1, HL2, HL3: (no value), led:LED5MM
- added IC1: 24LC256SN, microchip:24LC256SN
- added JMEM: (no value), ArduinoBASIC:PINHD-1X4
- added L1: 100uh, rcl:L-US0207/10
- added L2: (no value), rcl:L-US0204/5
- added PINV: (no value), ArduinoBASIC:FE12-1
- added R10: 1, rcl:R-EU_M1206
- added R11: 180, rcl:R-EU_M1206
- added R12: 1k, rcl:R-EU_M0805
- added R13: 3k, rcl:R-EU_M0805
- added R2, R4, R6, R7, R8, R9: 10k, rcl:R-EU_R0805
- added R3, R5: 10k, rcl:R-EU_R1206W
- added SW1: POW, ArduinoBASIC:9077-2
- added T1, T2, T3: (no value), transistor:BC368-NPN-TO92-ECB
- added VD1: SS12, diode:SCHOTTKY-DIODESMD
- C2, C3: value 100n -> 1n; device rcl:C-EUC0805 -> rcl:C-EU025-025X050
- renumbered PORT1 to PING
Connections:
- new net N$10: SW11.O, SW12.O
- new net N$11: HL1.C, T1.C
- new net N$12: R2.2, T1.B
- new net N$13: HL1.A, R3.1
- new net N$14: HL2.C, T2.C
- new net N$15: R4.2, T2.B
- new net N$16: HL2.A, R5.1
- new net N$17: HL3.C, T3.C
- new net N$18: R6.2, T3.B
- new net N$19: HL3.A, R7.1
- new net N$21: C10.2, C9.+, L2.1, R13.2, VD1.C
- new net N$4: POW.1, SW11.P, SW12.P
- net AREF: now also C1.2; no longer C2.2
- net D14: no longer S33.S
- net D15: no longer S21.S1
- net D4: now also PORT.1, R2.1; no longer PORT.3
- net D6: now also PORT.2, R4.1; no longer PORT.1
- net D7: now also PORT.3, R6.1; no longer PORT.2
- net GND: now also C1.1, C10.1, C11.1, C12.-, C3.1, C4.2, C5.2, C6.2, C7.2, C8.-, C9.-, IC1.A0, IC1.A1, IC1.A2, IC1.GND, IC1.WP, JMEM.4, R12.1, T1.E, T2.E, T3.E; no longer 3C10.-, 3C11.-, 3C12.1, 3C6.1, 3C7.1, 3C8.2, 3C9.2, 3R8.1, C1.2, C3.2
- net N$1: now also C2.2; no longer 3C6.2
- net N$2: now also C3.2; no longer 3C7.2
- net N$3: now also C7.1, C8.+, R10.1, SW11.S, SW12.S; no longer 3C10.+, 3C8.1, 3R6.1, POW.1
- net N$5: now also R11.1; no longer 3R5.1
- net N$6: now also L1.1, R10.2, R11.2; no longer 3L2.1, 3R5.2, 3R6.2
- net N$7: now also R12.2, R13.1; no longer 3R7.1, 3R8.2
- net N$8: now also L1.2, VD1.A; no longer 3L2.2, 3VD2.A
- net N$9: now also C6.1; no longer 3C9.1
- net SCL: now also IC1.SDA, JMEM.1, R9.1
- net SDA: now also IC1.SCL, JMEM.2, R8.1
- net U6: no longer S21.P1
- net VCC: now also C11.2, C12.+, C4.1, C5.1, IC1.VCC, JMEM.3, L2.2, PINV.1, PINV.10, PINV.11, PINV.12, PINV.2, PINV.3, PINV.4, PINV.5, PINV.6, PINV.7, PINV.8, PINV.9, R3.2, R5.2, R7.2, R8.2, R9.2; no longer 3C11.+, 3C12.2, 3R7.2, 3VD2.C, C1.1, C3.1
Other:
- moved on the sheet: C1, C2, C3, DA1, ISP, KB1, KB2, POW, S1, S10, S11, S12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
