File: aduinobasic.sch (EAGLE design)
At the start: 106 parts, among them IC1 24LC256SN, SW1 POW

Commit message: .
Parts:
- HL1, HL2, HL3: device led:LED5MM -> ArduinoBASIC:LED5MM
- R2: value 10k -> 1k
- renumbered IC1 to DD2
Changed lines of the file:
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@@
 <part name="SW1" library="ArduinoBASIC" deviceset="9077-2" device="" value="POW"/>
 <part name="GND1" library="supply1" deviceset="GND" device=""/>
-<part name="IC1" library="microchip" deviceset="24*" device="SN" technology="LC256"/>
+<part name="DD2" library="microchip" deviceset="24*" device="SN" technology="LC256"/>
 <part name="R8" library="rcl" deviceset="R-EU_" device="R0805" value="10k"/>
 <part name="GND12" library="supply1" deviceset="GND" device=""/>
@@
 <part name="GND14" library="supply1" deviceset="GND" device=""/>
 <part name="P+5" library="supply1" deviceset="VCC" device=""/>
-<part name="HL1" library="led" deviceset="LED" device="5MM"/>
+<part name="HL1" library="ArduinoBASIC" deviceset="LED" device="5MM"/>
 <part name="PINV" library="ArduinoBASIC" deviceset="FE12-1" device="">
 <attribute name="MF" value=""/>
@@
 <part name="R3" library="rcl" deviceset="R-EU_" device="R1206W" value="10k"/>
 <part name="GND15" library="supply1" deviceset="GND" device=""/>
-<part name="R2" library="rcl" deviceset="R-EU_" device="R0805" value="10k"/>
+<part name="R2" library="rcl" deviceset="R-EU_" device="R0805" value="1k"/>
 <part name="P+8" library="supply1" deviceset="VCC" device=""/>
-<part name="HL2" library="led" deviceset="LED" device="5MM"/>
+<part name="HL2" library="ArduinoBASIC" deviceset="LED" device="5MM"/>
 <part name="T2" library="transistor" deviceset="*-NPN-" device="TO92-ECB" technology="BC368"/>
 <part name="R5" library="rcl" deviceset="R-EU_" device="R1206W" value="10k"/>
@@
 <part name="R4" library="rcl" deviceset="R-EU_" device="R0805" value="10k"/>
 <part name="P+9" library="supply1" deviceset="VCC" device=""/>
-<part name="HL3" library="led" deviceset="LED" device="5MM"/>
+<part name="HL3" library="ArduinoBASIC" deviceset="LED" device="5MM"/>
 <part name="T3" library="transistor" deviceset="*-NPN-" device="TO92-ECB" technology="BC368"/>
 <part name="R7" library="rcl" deviceset="R-EU_" device="R0805" value="10k"/>
@@
 <instance part="SW1" gate="2" x="185.42" y="132.08" rot="R270"/>
 <instance part="GND1" gate="1" x="177.8" y="114.3"/>
-<instance part="IC1" gate="G$1" x="193.04" y="165.1"/>
+<instance part="DD2" gate="G$1" x="193.04" y="165.1"/>
 <instance part="R8" gate="G$1" x="177.8" y="180.34" rot="R90"/>
 <instance part="GND12" gate="1" x="200.66" y="149.86"/>
@@
 </instance>
 <instance part="T1" gate="G$1" x="45.72" y="185.42"/>
-<instance part="R3" gate="G$1" x="55.88" y="195.58" rot="R270"/>
+<instance part="R3" gate="G$1" x="55.88" y="195.58" smashed="yes" rot="R270">
+<attribute name="NAME" x="57.3786" y="199.39" size="1.778" layer="95" rot="R270"/>
+<attribute name="VALUE" x="52.578" y="199.39" size="1.778" layer="96" rot="R270"/>
+</instance>
 <instance part="GND15" gate="1" x="48.26" y="175.26"/>
-<instance part="R2" gate="G$1" x="40.64" y="193.04" rot="R270"/>
+<instance part="R2" gate="G$1" x="40.64" y="193.04" smashed="yes" rot="R270">
+<attribute name="NAME" x="42.1386" y="196.85" size="1.778" layer="95" rot="R270"/>
+<attribute name="VALUE" x="37.338" y="196.85" size="1.778" layer="96" rot="R270"/>
+</instance>
 <instance part="P+8" gate="VCC" x="55.88" y="185.42" smashed="yes" rot="R180">
 <attribute name="VALUE" x="53.34" y="182.88" size="1.778" layer="96"/>
@@
 <instance part="HL2" gate="G$1" x="71.12" y="198.12"/>
 <instance part="T2" gate="G$1" x="68.58" y="185.42"/>
-<instance part="R5" gate="G$1" x="78.74" y="195.58" rot="R270"/>
+<instance part="R5" gate="G$1" x="78.74" y="195.58" smashed="yes" rot="R270">
+<attribute name="NAME" x="80.2386" y="199.39" size="1.778" layer="95" rot="R270"/>
+<attribute name="VALUE" x="75.438" y="199.39" size="1.778" layer="96" rot="R270"/>
+</instance>
 <instance part="GND16" gate="1" x="71.12" y="175.26"/>
-<instance part="R4" gate="G$1" x="63.5" y="193.04" rot="R270"/>
+<instance part="R4" gate="G$1" x="63.5" y="193.04" smashed="yes" rot="R270">
+<attribute name="NAME" x="64.9986" y="196.85" size="1.778" layer="95" rot="R270"/>
+<attribute name="VALUE" x="60.198" y="196.85" size="1.778" layer="96" rot="R270"/>
+</instance>
 <instance part="P+9" gate="VCC" x="78.74" y="185.42" smashed="yes" rot="R180">
 <attribute name="VALUE" x="76.2" y="182.88" size="1.778" layer="96"/>
@@
 <instance part="HL3" gate="G$1" x="96.52" y="198.12"/>
 <instance part="T3" gate="G$1" x="93.98" y="185.42"/>
-<instance part="R7" gate="G$1" x="104.14" y="195.58" rot="R270"/>
+<instance part="R7" gate="G$1" x="104.14" y="195.58" smashed="yes" rot="R270">
+<attribute name="NAME" x="105.6386" y="199.39" size="1.778" layer="95" rot="R270"/>
+<attribute name="VALUE" x="100.838" y="199.39" size="1.778" layer="96" rot="R270"/>
+</instance>
 <instance part="GND17" gate="1" x="96.52" y="175.26"/>
-<instance part="R6" gate="G$1" x="88.9" y="193.04" rot="R270"/>
+<instance part="R6" gate="G$1" x="88.9" y="193.04" smashed="yes" rot="R270">
+<attribute name="NAME" x="90.3986" y="196.85" size="1.778" layer="95" rot="R270"/>
+<attribute name="VALUE" x="85.598" y="196.85" size="1.778" layer="96" rot="R270"/>
+</instance>
 <instance part="P+10" gate="VCC" x="104.14" y="185.42" smashed="yes" rot="R180">
 <attribute name="VALUE" x="101.6" y="182.88" size="1.778" layer="96"/>
@@
 </segment>
 <segment>
-<pinref part="IC1" gate="G$1" pin="GND"/>
+<pinref part="DD2" gate="G$1" pin="GND"/>
 <pinref part="GND12" gate="1" pin="GND"/>
 <wire x1="200.66" y1="154.94" x2="200.66" y2="152.4" width="0.1524" layer="91"/>
 </segment>
 <segment>
-<pinref part="IC1" gate="G$1" pin="A0"/>
+<pinref part="DD2" gate="G$1" pin="A0"/>
 <wire x1="180.34" y1="160.02" x2="177.8" y2="160.02" width="0.1524" layer="91"/>
 <wire x1="177.8" y1="160.02" x2="177.8" y2="162.56" width="0.1524" layer="91"/>
-<pinref part="IC1" gate="G$1" pin="A1"/>
+<pinref part="DD2" gate="G$1" pin="A1"/>
 <wire x1="177.8" y1="162.56" x2="180.34" y2="162.56" width="0.1524" layer="91"/>
-<pinref part="IC1" gate="G$1" pin="A2"/>
+<pinref part="DD2" gate="G$1" pin="A2"/>
 <wire x1="180.34" y1="165.1" x2="177.8" y2="165.1" width="0.1524" layer="91"/>
 <wire x1="177.8" y1="165.1" x2="177.8" y2="162.56" width="0.1524" layer="91"/>
-<pinref part="IC1" gate="G$1" pin="WP"/>
+<pinref part="DD2" gate="G$1" pin="WP"/>
 <wire x1="180.34" y1="170.18" x2="177.8" y2="170.18" width="0.1524" layer="91"/>
 <wire x1="177.8" y1="170.18" x2="177.8" y2="165.1" width="0.1524" layer="91"/>
@@
 <wire x1="210.82" y1="190.5" x2="210.82" y2="187.96" width="0.1524" layer="91"/>
 <junction x="210.82" y="187.96"/>
-<pinref part="IC1" gate="G$1" pin="VCC"/>
+<pinref part="DD2" gate="G$1" pin="VCC"/>
 <wire x1="200.66" y1="177.8" x2="200.66" y2="187.96" width="0.1524" layer="91"/>
 <junction x="200.66" y="187.96"/>
@@
 </segment>
 <segment>
-<pinref part="IC1" gate="G$1" pin="SCL"/>
+<pinref part="DD2" gate="G$1" pin="SCL"/>
 <wire x1="180.34" y1="172.72" x2="177.8" y2="172.72" width="0.1524" layer="91"/>
 <pinref part="R8" gate="G$1" pin="1"/>
@@
 </segment>
 <segment>
-<pinref part="IC1" gate="G$1" pin="SDA"/>
+<pinref part="DD2" gate="G$1" pin="SDA"/>
 <wire x1="208.28" y1="165.1" x2="210.82" y2="165.1" width="0.1524" layer="91"/>
 <pinref part="R9" gate="G$1" pin="1"/>
@@
 <pinref part="R2" gate="G$1" pin="1"/>
 <wire x1="40.64" y1="198.12" x2="40.64" y2="203.2" width="0.1524" layer="91"/>
-<label x="38.1" y="200.66" size="1.778" layer="95" rot="R180"/>
+<label x="40.64" y="200.66" size="1.778" layer="95" rot="R90"/>
 </segment>
 </net>
@@
 <pinref part="R4" gate="G$1" pin="1"/>
 <wire x1="63.5" y1="198.12" x2="63.5" y2="203.2" width="0.1524" layer="91"/>
-<label x="58.42" y="200.66" size="1.778" layer="95"/>
+<label x="63.5" y="200.66" size="1.778" layer="95" rot="R90"/>
 </segment>
 </net>
@@
 <pinref part="R6" gate="G$1" pin="1"/>
 <wire x1="88.9" y1="198.12" x2="88.9" y2="203.2" width="0.1524" layer="91"/>
-<label x="83.82" y="200.66" size="1.778" layer="95"/>
-</segment>
-</net>
+<label x="88.9" y="200.66" size="1.778" layer="95" rot="R90"/>
+</segment>
+</net>

Commit message: .
Parts:
- added KB3, KB4: (no value), pinhead:PINHD-1X1
- renumbered T1 to VT1, T2 to VT2, T3 to VT3
Connections:
- net GND: now also KB4.1
- net VCC: now also KB3.1
Changed lines of the file:
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@@
 </part>
 <part name="P+7" library="supply1" deviceset="VCC" device=""/>
-<part name="T1" library="transistor" deviceset="*-NPN-" device="TO92-ECB" technology="BC368"/>
+<part name="VT1" library="transistor" deviceset="*-NPN-" device="TO92-ECB" technology="BC368"/>
 <part name="R3" library="rcl" deviceset="R-EU_" device="R1206W" value="10k"/>
 <part name="GND15" library="supply1" deviceset="GND" device=""/>
@@
 <part name="P+8" library="supply1" deviceset="VCC" device=""/>
 <part name="HL2" library="ArduinoBASIC" deviceset="LED" device="5MM"/>
-<part name="T2" library="transistor" deviceset="*-NPN-" device="TO92-ECB" technology="BC368"/>
+<part name="VT2" library="transistor" deviceset="*-NPN-" device="TO92-ECB" technology="BC368"/>
 <part name="R5" library="rcl" deviceset="R-EU_" device="R1206W" value="10k"/>
 <part name="GND16" library="supply1" deviceset="GND" device=""/>
@@
 <part name="P+9" library="supply1" deviceset="VCC" device=""/>
 <part name="HL3" library="ArduinoBASIC" deviceset="LED" device="5MM"/>
-<part name="T3" library="transistor" deviceset="*-NPN-" device="TO92-ECB" technology="BC368"/>
+<part name="VT3" library="transistor" deviceset="*-NPN-" device="TO92-ECB" technology="BC368"/>
 <part name="R7" library="rcl" deviceset="R-EU_" device="R0805" value="10k"/>
 <part name="GND17" library="supply1" deviceset="GND" device=""/>
@@
 <part name="C11" library="rcl" deviceset="C-EU" device="C1206" value="100n"/>
 <part name="GND19" library="supply1" deviceset="GND" device=""/>
+<part name="KB3" library="pinhead" deviceset="PINHD-1X1" device=""/>
+<part name="KB4" library="pinhead" deviceset="PINHD-1X1" device=""/>
+<part name="P+11" library="supply1" deviceset="VCC" device=""/>
+<part name="GND20" library="supply1" deviceset="GND" device=""/>
 </parts>
 <sheets>
@@
 <attribute name="VALUE" x="162.56" y="142.24" size="1.778" layer="96" rot="R180"/>
 </instance>
-<instance part="T1" gate="G$1" x="45.72" y="185.42"/>
+<instance part="VT1" gate="G$1" x="45.72" y="185.42"/>
 <instance part="R3" gate="G$1" x="55.88" y="195.58" smashed="yes" rot="R270">
 <attribute name="NAME" x="57.3786" y="199.39" size="1.778" layer="95" rot="R270"/>
@@
 </instance>
 <instance part="HL2" gate="G$1" x="71.12" y="198.12"/>
-<instance part="T2" gate="G$1" x="68.58" y="185.42"/>
+<instance part="VT2" gate="G$1" x="68.58" y="185.42"/>
 <instance part="R5" gate="G$1" x="78.74" y="195.58" smashed="yes" rot="R270">
 <attribute name="NAME" x="80.2386" y="199.39" size="1.778" layer="95" rot="R270"/>
@@
 </instance>
 <instance part="HL3" gate="G$1" x="96.52" y="198.12"/>
-<instance part="T3" gate="G$1" x="93.98" y="185.42"/>
+<instance part="VT3" gate="G$1" x="93.98" y="185.42"/>
 <instance part="R7" gate="G$1" x="104.14" y="195.58" smashed="yes" rot="R270">
 <attribute name="NAME" x="105.6386" y="199.39" size="1.778" layer="95" rot="R270"/>
@@
 </instance>
 <instance part="GND19" gate="1" x="264.16" y="104.14"/>
+<instance part="KB3" gate="G$1" x="127" y="195.58"/>
+<instance part="KB4" gate="G$1" x="127" y="185.42"/>
+<instance part="P+11" gate="VCC" x="114.3" y="200.66" smashed="yes">
+<attribute name="VALUE" x="116.84" y="203.2" size="1.778" layer="96" rot="R180"/>
+</instance>
+<instance part="GND20" gate="1" x="114.3" y="180.34"/>
 </instances>
 <busses>
@@
 </segment>
 <segment>
-<pinref part="T1" gate="G$1" pin="E"/>
+<pinref part="VT1" gate="G$1" pin="E"/>
 <pinref part="GND15" gate="1" pin="GND"/>
 <wire x1="48.26" y1="180.34" x2="48.26" y2="177.8" width="0.1524" layer="91"/>
 </segment>
 <segment>
-<pinref part="T2" gate="G$1" pin="E"/>
+<pinref part="VT2" gate="G$1" pin="E"/>
 <pinref part="GND16" gate="1" pin="GND"/>
 <wire x1="71.12" y1="180.34" x2="71.12" y2="177.8" width="0.1524" layer="91"/>
 </segment>
 <segment>
-<pinref part="T3" gate="G$1" pin="E"/>
+<pinref part="VT3" gate="G$1" pin="E"/>
 <pinref part="GND17" gate="1" pin="GND"/>
 <wire x1="96.52" y1="180.34" x2="96.52" y2="177.8" width="0.1524" layer="91"/>
@@
 <pinref part="GND19" gate="1" pin="GND"/>
 <wire x1="264.16" y1="109.22" x2="264.16" y2="106.68" width="0.1524" layer="91"/>
+</segment>
+<segment>
+<pinref part="KB4" gate="G$1" pin="1"/>
+<wire x1="124.46" y1="185.42" x2="114.3" y2="185.42" width="0.1524" layer="91"/>
+<pinref part="GND20" gate="1" pin="GND"/>
+<wire x1="114.3" y1="182.88" x2="114.3" y2="185.42" width="0.1524" layer="91"/>
 </segment>
 </net>
@@
 <junction x="276.86" y="119.38"/>
 </segment>
+<segment>
+<pinref part="KB3" gate="G$1" pin="1"/>
+<wire x1="124.46" y1="195.58" x2="114.3" y2="195.58" width="0.1524" layer="91"/>
+<pinref part="P+11" gate="VCC" pin="VCC"/>
+<wire x1="114.3" y1="198.12" x2="114.3" y2="195.58" width="0.1524" layer="91"/>
+</segment>
 </net>
 <net name="SCK" class="0">
@@
 <segment>
 <pinref part="HL1" gate="G$1" pin="C"/>
-<pinref part="T1" gate="G$1" pin="C"/>
+<pinref part="VT1" gate="G$1" pin="C"/>
 <wire x1="48.26" y1="193.04" x2="48.26" y2="190.5" width="0.1524" layer="91"/>
 </segment>
@@
 <segment>
 <pinref part="R2" gate="G$1" pin="2"/>
-<pinref part="T1" gate="G$1" pin="B"/>
+<pinref part="VT1" gate="G$1" pin="B"/>
 <wire x1="40.64" y1="187.96" x2="40.64" y2="185.42" width="0.1524" layer="91"/>
 <wire x1="40.64" y1="185.42" x2="43.18" y2="185.42" width="0.1524" layer="91"/>
@@
 <segment>
 <pinref part="HL2" gate="G$1" pin="C"/>
-<pinref part="T2" gate="G$1" pin="C"/>
+<pinref part="VT2" gate="G$1" pin="C"/>
 <wire x1="71.12" y1="193.04" x2="71.12" y2="190.5" width="0.1524" layer="91"/>
 </segment>
@@
 <segment>
 <pinref part="R4" gate="G$1" pin="2"/>
-<pinref part="T2" gate="G$1" pin="B"/>
+<pinref part="VT2" gate="G$1" pin="B"/>
 <wire x1="63.5" y1="187.96" x2="63.5" y2="185.42" width="0.1524" layer="91"/>
 <wire x1="63.5" y1="185.42" x2="66.04" y2="185.42" width="0.1524" layer="91"/>
@@
 <segment>
 <pinref part="HL3" gate="G$1" pin="C"/>
-<pinref part="T3" gate="G$1" pin="C"/>
+<pinref part="VT3" gate="G$1" pin="C"/>
 <wire x1="96.52" y1="193.04" x2="96.52" y2="190.5" width="0.1524" layer="91"/>
 </segment>
@@
 <segment>
 <pinref part="R6" gate="G$1" pin="2"/>
-<pinref part="T3" gate="G$1" pin="B"/>
+<pinref part="VT3" gate="G$1" pin="B"/>
 <wire x1="91.44" y1="185.42" x2="88.9" y2="185.42" width="0.1524" layer="91"/>
 <wire x1="88.9" y1="185.42" x2="88.9" y2="187.96" width="0.1524" layer="91"/>

Commit message: .
Parts:
- added BUZ: (no value), pinhead:PINHD-1X1
- VT1, VT2, VT3: value (none) -> КТ315Б
Connections:
- net BUZ: now also BUZ.1
Other:
- note removed: "10 26"
- moved on the sheet: HL1, HL2, HL3, KB1, KB2, KB3, KB4, R2, R3, R4, R5, R6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

Commit message: .
Parts:
- R11: value 180 -> 200
Changed lines of the file:
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@@
 <part name="C7" library="rc-elektronik" deviceset="C-EU" device="C1206" value="100n"/>
 <part name="DA1" library="mc34063" deviceset="MC34063" device="AD"/>
-<part name="R11" library="rcl" deviceset="R-EU_" device="M1206" value="180"/>
+<part name="R11" library="rcl" deviceset="R-EU_" device="M1206" value="200"/>
 <part name="R10" library="rcl" deviceset="R-EU_" device="M1206" value="1"/>
 <part name="GND4" library="supply1" deviceset="GND" device=""/>
